File: hw/lse2_board/lse2_board.kicad_pcb (KiCad board)
At the start: 2 copper layers, 93.7 x 91.1 mm, 30 parts, among them IC1 DIGIT_DRIVER, IC2 DIGIT_DRIVER, J1 Conn_02x10_Odd_Even, J10 Conn_01x02, J2 Conn_02x10_Odd_Even, J3 Conn_02x10_Odd_Even, J4 Conn_02x10_Odd_Even, J5 Conn_02x03_Odd_Even, J6 Conn_01x03, J7 RF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

Commit message: v2
Parts:
- removed J6: Conn_01x03, Connector_PinSocket_2.54mm:PinSocket_1x03_P2.54mm_Vertical
- added R10: R, Resistor_SMD:R_1206_3216Metric, B.Cu at (132.7, 99.2)
- added R11: R, Resistor_SMD:R_1206_3216Metric, B.Cu at (133.2, 85.8)
- added R12: R, Resistor_SMD:R_1206_3216Metric, B.Cu at (129.0, 82.8)
- added R13: R, Resistor_SMD:R_1206_3216Metric, B.Cu at (146.6, 91.3)
- added R14: R, Resistor_SMD:R_1206_3216Metric, B.Cu at (142.9, 99.2)
- added R15: R, Resistor_SMD:R_1206_3216Metric, B.Cu at (135.7, 99.2)
- added R16: R, Resistor_SMD:R_1206_3216Metric, B.Cu at (139.3, 99.1)
- added R17: R, Resistor_SMD:R_1206_3216Metric, B.Cu at (146.3, 99.2)
- added R18: R, Resistor_SMD:R_1206_3216Metric, B.Cu at (149.5, 85.2)
- added R19: R, Resistor_SMD:R_1206_3216Metric, B.Cu at (147.1, 82.1)
- added R6: R, Resistor_SMD:R_1206_3216Metric, B.Cu at (125.8, 94.0)
- added R7: R, Resistor_SMD:R_1206_3216Metric, B.Cu at (127.8, 91.0)
- added R8: R, Resistor_SMD:R_1206_3216Metric, B.Cu at (126.6, 99.2)
- added R9: R, Resistor_SMD:R_1206_3216Metric, B.Cu at (129.7, 99.2)
- added U1: NRF24L01_Breakout, RF_Module:nRF24L01_Breakout, F.Cu at (131.7, 60.7)
- C5, IC1: moved to B.Cu
- J5, J9: value Conn_02x03_Odd_Even -> Conn_02x05_Odd_Even; footprint Connector_PinHeader_2.54mm:PinHeader_2x03_P2.54mm_Vertical -> Connector_PinHeader_2.54mm:PinHeader_2x05_P2.54mm_Vertical
- J7: value RF -> Conn_01x05; footprint Connector_PinHeader_2.54mm:PinHeader_2x04_P2.54mm_Vertical -> Connector_PinHeader_2.54mm:PinHeader_1x05_P2.54mm_Vertical
- moved J7 84.4 mm to (104.3, 66.0)
- moved C2 82.6 mm to (128.1, 58.8)
- moved J9 81.2 mm to (178.0, 76.4)
- moved IC1 63.6 mm to (116.3, 89.5), turned to 90 degrees
- moved C4 55.1 mm to (116.3, 95.9), turned to -90 degrees
- moved 3V3 54.2 mm to (110.9, 71.9), turned to -90 degrees
- moved GND 53.3 mm to (110.9, 77.6), turned to -90 degrees
- moved C1 50.7 mm to (122.4, 69.3), turned to 90 degrees
- moved IC2 48.8 mm to (160.8, 89.4), turned to 90 degrees
- moved J5 48.3 mm to (92.7, 76.4)
- moved C5 47.9 mm to (163.5, 89.9)
- moved D3 39.1 mm to (101.3, 88.6)
- moved J10 38.9 mm to (134.6, 82.6), turned to 90 degrees
- moved R2 38.8 mm to (122.4, 80.9), turned to -90 degrees
- moved D2 38.3 mm to (122.4, 76.1), turned to 90 degrees
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Connections:
- IC1 pad 10: Net-(DS1-B_CATHODE_NO.1) -> Net-(IC1-QB)
- IC1 pad 11: Net-(DS1-C_CATHODE_NO.1) -> Net-(IC1-QC)
- IC1 pad 12: Net-(DS1-D_CATHODE_NO.1) -> Net-(IC1-QD)
- IC1 pad 13: Net-(DS1-E_CATHODE_NO.1) -> Net-(IC1-QE)
- IC1 pad 14: Net-(DS1-G_CATHODE_NO.1) -> Net-(IC1-QG)
- IC1 pad 15: Net-(DS1-F_CATHODE_NO.1) -> Net-(IC1-QF)
- IC1 pad 7: CA/CC -> GND
- IC1 pad 9: Net-(DS1-A_CATHODE_NO.1) -> Net-(IC1-QA)
- IC2 pad 10: Net-(DS1-B_CATHODE_NO.2) -> Net-(IC2-QB)
- IC2 pad 11: Net-(DS1-C_CATHODE_NO.2) -> Net-(IC2-QC)
- IC2 pad 12: Net-(DS1-D_CATHODE_NO.2) -> Net-(IC2-QD)
- IC2 pad 13: Net-(DS1-E_CATHODE_NO.2) -> Net-(IC2-QE)
- IC2 pad 14: Net-(DS1-G_CATHODE_NO.2) -> Net-(IC2-QG)
- IC2 pad 15: Net-(DS1-F_CATHODE_NO.2) -> Net-(IC2-QF)
- IC2 pad 7: CA/CC -> GND
- IC2 pad 9: Net-(DS1-A_CATHODE_NO.2) -> Net-(IC2-QA)
- J1 pad 10: unconnected-(J1-Pin_10-Pad10) -> D0_L
- J1 pad 11: MISO_R -> MISO_L
- J1 pad 12: unconnected-(J1-Pin_12-Pad12) -> D3_L
- J1 pad 13: SCLK_L -> SCLK_R
- J1 pad 15: unconnected-(J1-Pin_15-Pad15) -> D1_L
- J1 pad 18: unconnected-(J1-Pin_18-Pad18) -> D2_L
- J1 pad 20: unconnected-(J1-Pin_20-Pad20) -> IMU_PWR_ENABLE
- J1 pad 3: MOSI_R -> MOSI_L
- J1 pad 5: LED_R -> LED_G
- J1 pad 6: unconnected-(J1-Pin_6-Pad6) -> LED_R
- J1 pad 7: LED_G -> unconnected-(J1-Pin_7-Pad7)
- J1 pad 8: unconnected-(J1-Pin_8-Pad8) -> LED_B
- J1 pad 9: LED_B -> unconnected-(J1-Pin_9-Pad9)
- J2 pad 12: MOSI_L -> MOSI_R
- J2 pad 14: MISO_L -> MISO_R
- J2 pad 18: unconnected-(J2-Pin_18-Pad18) -> RF_CE
- J2 pad 2: unconnected-(J2-Pin_2-Pad2) -> GND
- J2 pad 3: unconnected-(J2-Pin_3-Pad3) -> SS_RF
- J3 pad 10: D1_L -> unconnected-(J3-Pin_10-Pad10)
- J3 pad 12: D3_L -> unconnected-(J3-Pin_12-Pad12)
- J3 pad 13: D0_L -> unconnected-(J3-Pin_13-Pad13)
- J3 pad 3: unconnected-(J3-Pin_3-Pad3) -> SS_R
- J3 pad 4: unconnected-(J3-Pin_4-Pad4) -> GND
- J3 pad 5: IMU_PWR_ENABLE -> unconnected-(J3-Pin_5-Pad5)
- J3 pad 6: CA/CC -> SS_L
- J3 pad 7: RF_CE -> unconnected-(J3-Pin_7-Pad7)
- J3 pad 8: SCLK_R -> SCLK_L
- J4 pad 2: unconnected-(J4-Pin_2-Pad2) -> GND
- J4 pad 7: D2_L -> unconnected-(J4-Pin_7-Pad7)
- J7 pad 1: GND -> MISO_RF
- J7 pad 2: RF_CE -> MOSI_RF
- J7 pad 4: MISO_RF -> SS_RF
- J7 pad 5: unconnected-(J7-Pin_5-Pad5) -> GND
Routing:
- net CA/CC: track 77.5 -> 0.00 mm, vias 1 -> 0
- net SS_L: track 0.00 -> 77.0 mm
- net D2_L: track 82.6 -> 9.56 mm, vias 2 -> 0
- net SCLK_L: track 25.4 -> 80.6 mm
- net SCLK_RF: track 97.8 -> 44.5 mm, vias 1 -> 0
- net MOSI_RF: track 102.8 -> 55.4 mm, vias 1 -> 0
- net SS_RF: track 0.00 -> 44.6 mm
- net MISO_R: track 36.4 -> 80.7 mm, vias 0 -> 2
- net MOSI_R: track 38.0 -> 82.4 mm, vias 0 -> 2
- net SDA: track 76.4 -> 32.6 mm
- net MISO_L: track 70.6 -> 31.8 mm
- net SCL: track 80.6 -> 45.0 mm, vias 0 -> 1
- net MOSI_L: track 67.1 -> 32.1 mm
- net D3_L: track 49.2 -> 14.2 mm, vias 1 -> 0
- net GND: track 72.0 -> 39.0 mm
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Other:
- board size 93.7 x 91.1 mm -> 93.7 x 51.8 mm
- board text added: "- LSE2 - Adrià Brú i Miquel Limón"
- board text added: "SS_L"
- board text added: "SS_R"
- board text added: "SS_RF"
- board text removed: "LSE2 - Adrià Brú i Miquel Limón"

Commit message: nova placa (cal revisar)
Changed lines of the file:
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@@
+	)
+	(segment
+		(start 108.235 59)
+		(end 108.235 60.714275)
+		(width 0.2)
+		(layer "B.Cu")
+		(net 47)
 	)
 	(segment
@@
 	)
 	(segment
-		(start 106.84 57.7)
-		(end 108.235 59.095)
-		(width 0.2)
-		(layer "B.Cu")
-		(net 47)
-	)
-	(segment
 		(start 140.1 66.9)
 		(end 146.9 66.9)
@@
 	)
 	(segment
-		(start 108.235 59.095)
-		(end 108.235 60.714275)
-		(width 0.2)
-		(layer "B.Cu")
-		(net 47)
-	)
-	(segment
 		(start 111.720725 64.2)
 		(end 129 64.2)
@@
 		(start 156.4 76.4)
 		(end 177.96 76.4)
+		(width 0.2)
+		(layer "B.Cu")
+		(net 47)
+	)
+	(segment
+		(start 106.84 57.7)
+		(end 108.235 59)
 		(width 0.2)
 		(layer "B.Cu")
@@
 		(polygon
 			(pts
-				(xy 70.500117 49.611733) (xy 193.000117 49.911733) (xy 193.600117 148.911733) (xy 67.800117 149.211733)
+				(xy 70.500117 49.611733) (xy 193.000117 49.911733) (xy 193.36751 110.531523) (xy 68.840626 110.828487)
 			)
 		)
@@
 		(polygon
 			(pts
-				(xy 73.100117 52.611733) (xy 190.800117 53.311733) (xy 191.500117 147.611733) (xy 76.400117 147.111733)
+				(xy 73.100117 52.611733) (xy 190.800117 53.311733) (xy 191.23238 111.543675) (xy 75.140447 111.039366)
 			)
 		)
