File: hw/lse2_board/lse2_board.kicad_sch (KiCad schematic)
At the start: 30 parts, among them IC1 DIGIT_DRIVER, IC2 DIGIT_DRIVER, J1 Conn_02x10_Odd_Even, J10 Conn_01x02, J2 Conn_02x10_Odd_Even, J3 Conn_02x10_Odd_Even, J4 Conn_02x10_Odd_Even, J5 Conn_02x03_Odd_Even, J6 Conn_01x03, J7 RF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

Commit message: v2
Parts:
- removed J5, J9: Conn_02x03_Odd_Even, Connector_PinHeader_2.54mm:PinHeader_2x03_P2.54mm_Vertical, symbol Connector_Generic:Conn_02x03_Odd_Even
- removed J6: Conn_01x03, Connector_PinSocket_2.54mm:PinSocket_1x03_P2.54mm_Vertical, symbol Connector_Generic:Conn_01x03
- removed J7: RF, Connector_PinHeader_2.54mm:PinHeader_2x04_P2.54mm_Vertical, symbol Connector_Generic:Conn_02x04_Counter_Clockwise
- added J5, J9: Conn_02x05_Odd_Even, Connector_PinHeader_2.54mm:PinHeader_2x05_P2.54mm_Vertical, symbol Connector_Generic:Conn_02x05_Odd_Even
- added J7: Conn_01x05, Connector_PinHeader_2.54mm:PinHeader_1x05_P2.54mm_Vertical, symbol Connector_Generic:Conn_01x05
- added R10, R11, R12, R13, R14, R15, R16, R17, R18, R19, R6, R7, R8, R9: R, Resistor_SMD:R_1206_3216Metric, symbol Device:R
- added U1: NRF24L01_Breakout, RF_Module:nRF24L01_Breakout, symbol RF:NRF24L01_Breakout
- renumbered 3V3_TP1 to 3V3, GND_TP1 to GND1
Connections:
- net +3.3V: now also U1.2 (VCC)
- net CA/CC: no longer IC1.7 (BL), IC2.7 (BL), J3.6 (Pin_6)
- net D0_L: now also J1.10 (Pin_10); no longer J3.13 (Pin_13)
- net D1_L: now also J1.15 (Pin_15); no longer J3.10 (Pin_10)
- net D2_L: now also J1.18 (Pin_18); no longer J4.7 (Pin_7)
- net D3_L: now also J1.12 (Pin_12); no longer J3.12 (Pin_12)
- net GND: now also IC1.7 (BL), IC2.7 (BL), J2.2 (Pin_2), J3.4 (Pin_4), J4.2 (Pin_2), J5.10 (Pin_10), J5.9 (Pin_9), J7.5 (Pin_5), J9.10 (Pin_10), J9.9 (Pin_9), U1.1 (GND)
- net IMU_PWR_ENABLE: now also J1.20 (Pin_20); no longer J3.5 (Pin_5)
- net LED_B: now also J1.8 (Pin_8); no longer J1.9 (Pin_9)
- net LED_G: now also J1.5 (Pin_5); no longer J1.7 (Pin_7)
- net LED_R: now also J1.6 (Pin_6); no longer J1.5 (Pin_5)
- net MISO_L: now also J1.11 (Pin_11), J5.3 (Pin_3), J5.4 (Pin_4); no longer J2.14 (Pin_14)
- net MISO_R: now also J2.14 (Pin_14), J9.3 (Pin_3), J9.4 (Pin_4); no longer J1.11 (Pin_11)
- net MISO_RF: now also J7.1 (Pin_1), U1.7 (MISO)
- net MOSI_L: now also J1.3 (Pin_3), J5.1 (Pin_1), J5.2 (Pin_2); no longer J2.12 (Pin_12)
- net MOSI_R: now also J2.12 (Pin_12), J9.1 (Pin_1), J9.2 (Pin_2); no longer J1.3 (Pin_3)
- net MOSI_RF: now also J7.2 (Pin_2), U1.6 (MOSI)
- net RF_CE: now also J2.18 (Pin_18), U1.3 (CE); no longer J3.7 (Pin_7)
- net SCLK_L: now also J3.8 (Pin_8), J5.5 (Pin_5), J5.6 (Pin_6); no longer J1.13 (Pin_13)
- net SCLK_R: now also J1.13 (Pin_13), J9.5 (Pin_5), J9.6 (Pin_6); no longer J3.8 (Pin_8)
- net SCLK_RF: now also J7.3 (Pin_3), U1.5 (SCK)
- net SS_R: now reaches J3.3 (Pin_3)
- net SS_R: now also J9.7 (Pin_7), J9.8 (Pin_8)
- net at DS1.10 (B_CATHODE_NO.2): now also R18.1; no longer IC2.10 (QB)
- net at IC2.11 (QC): now also R17.2; no longer DS1.8 (C_CATHODE_NO.2)
- net at IC2.12 (QD): now also R16.2; no longer DS1.6 (D_CATHODE_NO.2)
- net at DS1.5 (E_CATHODE_NO.2): now also R15.1; no longer IC2.13 (QE)
- net at IC2.14 (QG): now also R14.2; no longer DS1.7 (G_CATHODE_NO.2)
- net at IC2.15 (QF): now also R13.2; no longer DS1.12 (F_CATHODE_NO.2)
- net at IC2.9 (QA): now also R19.2; no longer DS1.11 (A_CATHODE_NO.2)
- net SS_RF: now reaches J2.3 (Pin_3)
- net SS_RF: now also J7.4 (Pin_4), U1.4 (~{CSN})
- net at DS1.1 (E_CATHODE_NO.1): now also R8.2; no longer IC1.13 (QE)
- net at DS1.15 (B_CATHODE_NO.1): now also R11.2; no longer IC1.10 (QB)
- net at DS1.16 (A_CATHODE_NO.1): now also R12.2; no longer IC1.9 (QA)
- net at IC1.14 (QG): now also R7.1; no longer DS1.17 (G_CATHODE_NO.1)
- net at IC1.15 (QF): now also R6.1; no longer DS1.18 (F_CATHODE_NO.1)
- net at DS1.2 (D_CATHODE_NO.1): now also R9.2; no longer IC1.12 (QD)
- net at IC1.11 (QC): now also R10.1; no longer DS1.3 (C_CATHODE_NO.1)
- new net: IC2.13 (QE), R15.2
- new net: DS1.18 (F_CATHODE_NO.1), R6.2
- new net: IC2.10 (QB), R18.2
- new net: DS1.17 (G_CATHODE_NO.1), R7.2
- new net: DS1.3 (C_CATHODE_NO.1), R10.2
- new net: DS1.11 (A_CATHODE_NO.2), R19.1
- new net: DS1.12 (F_CATHODE_NO.2), R13.1
- new net: DS1.6 (D_CATHODE_NO.2), R16.1
- new net: DS1.7 (G_CATHODE_NO.2), R14.1
- new net: DS1.8 (C_CATHODE_NO.2), R17.1
- new net: IC1.10 (QB), R11.1
- new net: IC1.12 (QD), R9.1
- new net: IC1.13 (QE), R8.1
- new net: IC1.9 (QA), R12.1
- new net SS_L: J3.6 (Pin_6), J5.7 (Pin_7), J5.8 (Pin_8)
- no-connect marks 60 -> 54
Other:
- moved on the sheet: C2, C4, D3, IC1, IC2, J10, R3, R4, R5

Commit message: nova placa (cal revisar)
Parts:
- removed 3V3, GND1: TestPoint, Connector_PinHeader_2.54mm:PinHeader_1x01_P2.54mm_Vertical, symbol Connector:TestPoint
- added J6: Conn_01x02, Connector_PinHeader_2.54mm:PinHeader_1x02_P2.54mm_Vertical, symbol Connector_Generic:Conn_01x02
Connections:
- net +3.3V: now also J6.1 (Pin_1)
- net GND: now also J6.2 (Pin_2)
Other:
- note added: "PWR test"
Changed lines of the file:
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@@
 		)
 	)
+	(text "PWR test"
+		(exclude_from_sim no)
+		(at 29.718 100.584 0)
+		(effects
+			(font
+				(size 1.27 1.27)
+			)
+		)
+	)
 	(text "Mòdul RF"
 		(exclude_from_sim no)
@@
 	)
 	(junction
-		(at 87.63 52.07)
-		(diameter 0)
-		(color 0 0 0 0)
-	)
-	(junction
 		(at 26.67 176.53)
 		(diameter 0)
 		(color 0 0 0 0)
 	)
-	(junction
-		(at 39.37 49.53)
-		(diameter 0)
-		(color 0 0 0 0)
-	)
 	(no_connect
 		(at 68.58 96.52)
@@
 	(wire
 		(pts
-			(xy 35.56 49.53) (xy 39.37 49.53)
+			(xy 35.56 49.53) (xy 45.72 49.53)
 		)
 		(stroke
@@
 	(wire
 		(pts
-			(xy 260.35 77.47) (xy 260.35 80.01)
+			(xy 21.59 107.95) (xy 29.21 107.95)
 		)
 		(stroke
@@
 	(wire
 		(pts
-			(xy 193.04 97.79) (xy 194.31 97.79)
+			(xy 260.35 77.47) (xy 260.35 80.01)
 		)
 		(stroke
@@
 	(wire
 		(pts
-			(xy 35.56 67.31) (xy 35.56 69.85)
+			(xy 193.04 97.79) (xy 194.31 97.79)
 		)
 		(stroke
@@
 	(wire
 		(pts
-			(xy 255.27 95.25) (xy 259.08 95.25)
+			(xy 35.56 67.31) (xy 35.56 69.85)
 		)
 		(stroke
@@
 	(wire
 		(pts
-			(xy 39.37 49.53) (xy 45.72 49.53)
+			(xy 255.27 95.25) (xy 259.08 95.25)
 		)
 		(stroke
@@
 	(wire
 		(pts
-			(xy 99.06 52.07) (xy 87.63 52.07)
+			(xy 81.28 52.07) (xy 99.06 52.07)
 		)
 		(stroke
@@
 	(wire
 		(pts
-			(xy 87.63 52.07) (xy 81.28 52.07)
-		)
-		(stroke
-			(width 0)
-			(type default)
-		)
-	)
-	(wire
-		(pts
 			(xy 231.14 144.78) (xy 231.14 146.05)
 		)
@@
 	(wire
 		(pts
+			(xy 21.59 105.41) (xy 29.21 105.41)
+		)
+		(stroke
+			(width 0)
+			(type default)
+		)
+	)
+	(wire
+		(pts
 			(xy 273.05 44.45) (xy 273.05 46.99)
 		)
@@
 	)
 	(symbol
-		(lib_id "Connector:TestPoint")
-		(at 87.63 52.07 0)
-		(unit 1)
-		(exclude_from_sim no)
-		(in_bom yes)
-		(on_board yes)
-		(dnp no)
-		(fields_autoplaced yes)
-		(property "Reference" "GND1"
-			(at 90.17 47.4979 0)
-			(effects
-				(font
-					(size 1.27 1.27)
-				)
-				(justify left)
-			)
-		)
-		(property "Value" "TestPoint"
-			(at 90.17 50.0379 0)
-			(effects
-				(font
-					(size 1.27 1.27)
-				)
-				(justify left)
-			)
-		)
-		(property "Footprint" "Connector_PinHeader_2.54mm:PinHeader_1x01_P2.54mm_Vertical"
-			(at 92.71 52.07 0)
-			(effects
-				(font
-					(size 1.27 1.27)
-				)
-				(hide yes)
-			)
-		)
-		(property "Datasheet" "~"
-			(at 92.71 52.07 0)
-			(effects
-				(font
-					(size 1.27 1.27)
-				)
-				(hide yes)
-			)
-		)
-		(property "Description" "test point"
-			(at 87.63 52.07 0)
-			(effects
-				(font
-					(size 1.27 1.27)
-				)
-				(hide yes)
-			)
-		)
-		(pin "1"
-		)
-		(instances
-			(project ""
-				(path "/45a51f49-1af1-447d-b599-00b362b8d1f6"
-					(reference "GND1")
-					(unit 1)
-				)
-			)
-		)
-	)
-	(symbol
 		(lib_id "power:GND")
 		(at 62.23 184.15 0)
@@
 	)
 	(symbol
-		(lib_id "Connector:TestPoint")
-		(at 39.37 49.53 0)
-		(unit 1)
-		(exclude_from_sim no)
-		(in_bom yes)
-		(on_board yes)
-		(dnp no)
-		(fields_autoplaced yes)
-		(property "Reference" "3V3"
-			(at 41.91 44.9579 0)
-			(effects
-				(font
-					(size 1.27 1.27)
-				)
-				(justify left)
-			)
-		)
-		(property "Value" "TestPoint"
-			(at 41.91 47.4979 0)
-			(effects
-				(font
-					(size 1.27 1.27)
-				)
-				(justify left)
-			)
-		)
-		(property "Footprint" "Connector_PinHeader_2.54mm:PinHeader_1x01_P2.54mm_Vertical"
-			(at 44.45 49.53 0)
-			(effects
-				(font
-					(size 1.27 1.27)
-				)
-				(hide yes)
-			)
-		)
-		(property "Datasheet" "~"
-			(at 44.45 49.53 0)
-			(effects
-				(font
-					(size 1.27 1.27)
-				)
-				(hide yes)
-			)
-		)
-		(property "Description" "test point"
-			(at 39.37 49.53 0)
-			(effects
-				(font
-					(size 1.27 1.27)
-				)
-				(hide yes)
-			)
-		)
-		(pin "1"
-		)
-		(instances
-			(project "lse2_board"
-				(path "/45a51f49-1af1-447d-b599-00b362b8d1f6"
-					(reference "3V3")
-					(unit 1)
-				)
-			)
-		)
-	)
-	(symbol
 		(lib_id "power:GND")
 		(at 161.29 180.34 0)
@@
 	)
 	(symbol
+		(lib_id "power:GND")
+		(at 21.59 107.95 0)
+		(unit 1)
+		(exclude_from_sim no)
+		(in_bom yes)
+		(on_board yes)
+		(dnp no)
+		(fields_autoplaced yes)
+		(property "Reference" "#PWR032"
+			(at 21.59 114.3 0)
+			(effects
+				(font
+					(size 1.27 1.27)
+				)
+				(hide yes)
+			)
+		)
+		(property "Value" "GND"
+			(at 21.59 113.03 0)
+			(effects
+				(font
+					(size 1.27 1.27)
+				)
+			)
+		)
+		(property "Footprint" ""
+			(at 21.59 107.95 0)
+			(effects
+				(font
+					(size 1.27 1.27)
+				)
+				(hide yes)
+			)
+		)
+		(property "Datasheet" ""
+			(at 21.59 107.95 0)
+			(effects
+				(font
+					(size 1.27 1.27)
+				)
+				(hide yes)
+			)
+		)
+		(property "Description" "Power symbol creates a global label with name \"GND\" , ground"
+			(at 21.59 107.95 0)
+			(effects
+				(font
+					(size 1.27 1.27)
+				)
+				(hide yes)
+			)
+		)
+		(pin "1"
+		)
+		(instances
+			(project "lse2_board"
+				(path "/45a51f49-1af1-447d-b599-00b362b8d1f6"
+					(reference "#PWR032")
+					(unit 1)
+				)
+			)
+		)
+	)
+	(symbol
 		(lib_id "Device:LED_RKGB")
 		(at 210.82 36.83 0)
@@
 	)
 	(symbol
+		(lib_id "power:+3.3V")
+		(at 21.59 105.41 0)
+		(unit 1)
+		(exclude_from_sim no)
+		(in_bom yes)
+		(on_board yes)
+		(dnp no)
+		(fields_autoplaced yes)
+		(property "Reference" "#PWR031"
+			(at 21.59 109.22 0)
+			(effects
+				(font
+					(size 1.27 1.27)
+				)
+				(hide yes)
+			)
+		)
+		(property "Value" "+3.3V"
+			(at 21.59 100.33 0)
+			(effects
+				(font
+					(size 1.27 1.27)
+				)
+			)
+		)
+		(property "Footprint" ""
+			(at 21.59 105.41 0)
+			(effects
+				(font
+					(size 1.27 1.27)
+				)
+				(hide yes)
+			)
+		)
+		(property "Datasheet" ""
+			(at 21.59 105.41 0)
+			(effects
+				(font
+					(size 1.27 1.27)
+				)
+				(hide yes)
+			)
+		)
+		(property "Description" "Power symbol creates a global label with name \"+3.3V\""
+			(at 21.59 105.41 0)
+			(effects
+				(font
+					(size 1.27 1.27)
+				)
+				(hide yes)
+			)
+		)
+		(pin "1"
+		)
+		(instances
+			(project "lse2_board"
+				(path "/45a51f49-1af1-447d-b599-00b362b8d1f6"
+					(reference "#PWR031")
+					(unit 1)
+				)
+			)
+		)
+	)
+	(symbol
 		(lib_id "power:GND")
 		(at 26.67 180.34 0)
@@
 					(unit 1)
 				)
+			)
+		)
+	)
+	(symbol
+		(lib_id "Connector_Generic:Conn_01x02")
+		(at 34.29 105.41 0)
+		(unit 1)
+		(exclude_from_sim no)
+		(in_bom yes)
+		(on_board yes)
+		(dnp no)
+		(fields_autoplaced yes)
+		(property "Reference" "J6"
+			(at 36.83 105.4099 0)
+			(effects
+				(font
+					(size 1.27 1.27)
+				)
+				(justify left)
+			)
+		)
+		(property "Value" "Conn_01x02"
+			(at 36.83 107.9499 0)
+			(effects
+				(font
+					(size 1.27 1.27)
+				)
+				(justify left)
+			)
+		)
+		(property "Footprint" "Connector_PinHeader_2.54mm:PinHeader_1x02_P2.54mm_Vertical"
+			(at 34.29 105.41 0)
+			(effects
+				(font
+					(size 1.27 1.27)
+				)
+				(hide yes)
+			)
+		)
+		(property "Datasheet" "~"
+			(at 34.29 105.41 0)
+			(effects
+				(font
+					(size 1.27 1.27)
+				)
+				(hide yes)
+			)
+		)
+		(property "Description" "Generic connector, single row, 01x02, script generated (kicad-library-utils/schlib/autogen/connector/)"
+			(at 34.29 105.41 0)
+			(effects
+				(font
+					(size 1.27 1.27)
+				)
+				(hide yes)
+			)
+		)
+		(pin "2"
+		)
+		(pin "1"
+		)
+		(instances
+			(project "lse2_board"
+				(path "/45a51f49-1af1-447d-b599-00b362b8d1f6"
+					(reference "J6")
+					(unit 1)
+				)
